File: pcb/ec-stingy/ec-stingy.kicad_sch (KiCad schematic)
At the start: 39 parts

Commit message: reconstructed schematic
Parts:
- removed C?: 3.3n, symbol Device:C
- removed R? (x2): 1Meg, symbol Device:R
- removed R?: 100k, symbol Device:R
- added C?: 1.5n, symbol Device:C
- added C? (x2): 0.33u, symbol Device:C
- added C?: 0.1u, symbol Device:C
- added R? (x4): 10Meg, symbol Device:R
- added R? (x2): 1Meg, symbol Device:R
- added R?: 1.4Meg, symbol Device:R
- C?: value 10p -> 0.33u
- C?: value 22n -> 10n
Connections:
- net +3.3V: now also U?.15 (FR), U?.17 (+VS), C?.1, R?.2
- net GND: now also U?.16 (GND), U?.PAD (GND_PAD), C?.1, C?.2, R?.2
- net at U?.6 (SW): now also C?.2, R?.2
- net at R?.2, U?.10 (OUT): now also C?.2
- net at U?.18 (REFIN): now also C?.2, R?.1, R?.1
- net at U?.19 (IAOUT): now also R?.2, R?.2
- net at C?.2, U?.20 (HPSENSE): now also R?.1
- net at C?.1, U?.7 (OPAMP+): now also R?.1
- net at C?.2, R?.1, U?.8 (REFOUT): now also C?.1
- new net: R?.1, R?.1, R?.2
- new net: C?.1, R?.1, R?.2
Other:
- moved on the sheet: C?
