File: pcb/ec-stingy/ec-stingy.kicad_sch (KiCad schematic)
At the start: 50 parts

Commit message: assigning footprints progress
Parts:
- added D1: LED, LED_SMD:LED_0603_1608Metric, symbol Device:LED
- added R1: 1k, symbol Device:R
- C1, C12, C7, C8, C9: renamed from C?; footprint (none) -> Capacitor_SMD:C_0603_1608Metric
- C10, C11, C20: renamed from C?; value 0.1u -> 100n; footprint (none) -> Capacitor_SMD:C_0402_1005Metric
- C13, C14, C15, C17, C2, C21, C22, C3, C4, C5, C6: renamed from C?; footprint (none) -> Capacitor_SMD:C_0402_1005Metric
- C16, C18, C19: renamed from C?; value 0.33u -> 330n; footprint (none) -> Capacitor_SMD:C_0402_1005Metric
- D2: renamed from D?; footprint (none) -> LED_SMD:LED_0603_1608Metric
- FB1: renamed from FB?; footprint (none) -> Inductor_SMD:L_0603_1608Metric
- J1: renamed from J?; footprint (none) -> Connector_USB:USB_Micro-B_Wuerth_629105150521
- J2: renamed from J?; footprint (none) -> Connector_PinHeader_2.54mm:PinHeader_1x04_P2.54mm_Vertical
- J4: renamed from J?; footprint (none) -> Connector_PinHeader_2.54mm:PinHeader_1x02_P2.54mm_Vertical
- gave numbers to parts that had none: 23
Connections:
- net +3.3V: now also U3.13 (~{SDN}), D1.2 (A)
- net GND: now also R1.2
- net RA: now reaches J3.R
- net RA: now also R6.2, R9.2
- net LA: now reaches J3.S
- net LA: now also R5.2, R7.2
- net RL: now reaches J3.T
- net RL: now also R13.2
- net HR_LED_K: now reaches D2.1 (K), R3.1
- net RLD: now reaches C17.2, R13.1, U3.5 (RLD)
- net HPSENSE: now reaches C16.2, R8.1, U3.20 (HPSENSE)
- net +IN: now reaches R7.1, U3.2 (+IN)
- net IAOUT: now reaches R10.2, R15.2, U3.19 (IAOUT)
- net REFIN: now reaches C18.2, R12.1, R14.1, U3.18 (REFIN)
- net USB_D-: now reaches J1.2 (D-), U2.5 (D-)
- net USB_D+: now reaches J1.3 (D+), U2.4 (D+)
- net HPDRIVE: now reaches C16.1, U3.1 (HPDRIVE)
- net -IN: now reaches R9.1, U3.3 (-IN)
- net RLDFB: now reaches C17.1, U3.4 (RLDFB)
- net SW: now reaches C19.2, R11.2, U3.6 (SW)
- net OPAMP+: now reaches C21.1, R16.1, U3.7 (OPAMP+)
- net REFOUT: now reaches C19.1, C21.2, R17.1, U3.8 (REFOUT)
- net OPAMP-: now reaches R17.2, R18.1, U3.9 (OPAMP-)
- new net PWR_LED_K: D1.1 (K), R1.1
- no-connect marks 11 -> 52
Other:
- note added: "1 x 100 nF per VDD pin"
- note added: "Bypass capacitor values taken directly from IC datasheet"
- note added: "CL = 2*(CL0-Cs) = 2*(10-5) pF = 10 pF"
- note added: "ECG front-end"
- note added: "Microcontroller"
- note added: "Oscillator"
- note added: "Pin-out using STM32CubeIDE"
- note added: "Power supply"
- note added: "See SPICE model & README for component value & circuitry details"
- note added: "USB-UART interface"
- note added: "ec-stingy"
- company: (none) -> Steve Farra
- title: (none) -> ec-stingy
- moved on the sheet: C1, C10, C11, C12, C13, C14, C15, C16, C17, C18, C19, C2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

Commit message: progress on layout
Parts:
- removed J1: USB_B_Micro, Connector_USB:USB_Micro-B_Wuerth_629105150521, symbol Connector:USB_B_Micro
- removed J3: AudioJack3, symbol Connector:AudioJack3
- removed SW1: SW_SPDT, symbol Switch:SW_SPDT
- added J1: PJ-320D-A, PJ-320D-A:HRO_PJ-320D-A, symbol PJ-320D-A:PJ-320D-A
- added J4: 105133-0011, 105133-0011:MOLEX_105133-0011, symbol 105133-0011:105133-0011
- added SW1: PCM12SMTR, PCM12SMTR:SW_PCM12SMTR, symbol PCM12SMTR:PCM12SMTR
- C12: renamed from C18; value 330n -> 100n
- R1: renamed from R5; footprint (none) -> Resistor_SMD:R_0603_1608Metric
- R10: renamed from R12; footprint (none) -> Resistor_SMD:R_0603_1608Metric
- R11: renamed from R14; footprint (none) -> Resistor_SMD:R_0603_1608Metric
- R12: renamed from R2; footprint (none) -> Resistor_SMD:R_0402_1005Metric
- R13: renamed from R10; footprint (none) -> Resistor_SMD:R_0603_1608Metric
- R14: renamed from R8; footprint (none) -> Resistor_SMD:R_0603_1608Metric
- R15: renamed from R11; footprint (none) -> Resistor_SMD:R_0603_1608Metric
- R16: renamed from R3; footprint (none) -> Resistor_SMD:R_0402_1005Metric
- R17: renamed from R1; footprint (none) -> Resistor_SMD:R_0402_1005Metric
- R18: renamed from R4; footprint (none) -> Resistor_SMD:R_0402_1005Metric
- R2: renamed from R15; footprint (none) -> Resistor_SMD:R_0603_1608Metric
- R3: renamed from R6; footprint (none) -> Resistor_SMD:R_0603_1608Metric
- R4: renamed from R16; footprint (none) -> Resistor_SMD:R_0603_1608Metric
- R5: renamed from R7; footprint (none) -> Resistor_SMD:R_0402_1005Metric
- R6: renamed from R9; footprint (none) -> Resistor_SMD:R_0402_1005Metric
- R7: renamed from R13; footprint (none) -> Resistor_SMD:R_0603_1608Metric
- R8: renamed from R17; footprint (none) -> Resistor_SMD:R_0402_1005Metric
- R9: renamed from R18; footprint (none) -> Resistor_SMD:R_0603_1608Metric
- U1: renamed from U3; footprint LFCSP_20 -> AD8232:LFCSP_20
- U3: renamed from U2; footprint Package_DFN_QFN:SiliconLabs_QFN-20-1EP_3x3mm_P0.5mm -> CP2102N-A02-GQFN20R:SILABS_CP2102N-A02-GQFN20R
- Y1: footprint (none) -> Crystal:Crystal_SMD_3225-4Pin_3.2x2.5mm
- renumbered C22 to C1, C20 to C10, C3 to C11, C4 to C13, C5 to C14, C19 to C15, C6 to C16, C7 to C17, C8 to C18, C9 to C19, C14 to C2, C10 to C20, C11 to C21, C12 to C22, C21 to C3, C17 to C4, C15 to C5, C16 to C6, C1 to C7, C13 to C8, C2 to C9, D2 to D1, D1 to D2, J4 to J2, J2 to J3, U1 to U2
Connections:
- net +3.3V: now also SW1.1
- net +5V: now also J4.1 (VBUS)
- net GND: now also J4.5 (GND), SW1.3
- net LA: now also J1.2
- net RA: now also J1.4
- net RL: now also J1.3
- net SW_BOOT0: now also SW1.2
- net USART2_RX: now also U2.17 (PA3); no longer U2.50 (PA15)
- net USB_D+: now also J4.3 (D+)
- net USB_D-: now also J4.2 (D-)
- new net: J4.S1 (SHIELD), J4.S2 (SHIELD), J4.S3 (SHIELD)
- new net: SW1.S1 (SHIELD), SW1.S2 (SHIELD), SW1.S3 (SHIELD), SW1.S4 (SHIELD)
- no-connect marks 52 -> 54

Commit message: more pcb progress
Parts:
- added H1, H2, H3, H4: MountingHole, MountingHole:MountingHole_2.2mm_M2, symbol Mechanical:MountingHole
Connections:
- net +IN renamed IN+
- net -IN renamed IN-
Other:
- note added: "M2"
- note added: "Mounting Holes"
Changed lines of the file:
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@@
+    (stroke (width 0) (type default) (color 0 0 0 0))
+  )
+  (polyline (pts (xy 321.31 194.31) (xy 321.31 222.25))
     (stroke (width 0) (type default) (color 0 0 0 0))
   )
@@
     (stroke (width 0) (type default) (color 0 0 0 0))
   )
+  (polyline (pts (xy 344.17 222.25) (xy 321.31 222.25))
+    (stroke (width 0) (type default) (color 0 0 0 0))
+  )
   (wire (pts (xy 240.03 76.2) (xy 254 76.2))
     (stroke (width 0) (type default) (color 0 0 0 0))
@@
     (stroke (width 0) (type default) (color 0 0 0 0))
   )
+  (polyline (pts (xy 344.17 194.31) (xy 344.17 222.25))
+    (stroke (width 0) (type default) (color 0 0 0 0))
+  )
   (wire (pts (xy 160.02 212.09) (xy 160.02 223.52))
     (stroke (width 0) (type default) (color 0 0 0 0))
@@
     (stroke (width 0) (type default) (color 0 0 0 0))
   )
+  (polyline (pts (xy 322.58 194.31) (xy 344.17 194.31))
+    (stroke (width 0) (type default) (color 0 0 0 0))
+  )
   (wire (pts (xy 227.33 96.52) (xy 251.46 96.52))
     (stroke (width 0) (type default) (color 0 0 0 0))
@@
   (wire (pts (xy 104.14 111.76) (xy 104.14 113.03))
     (stroke (width 0) (type default) (color 0 0 0 0))
+  )
+  (text "Mounting Holes" (at 320.04 193.04 0)
+    (effects (font (size 3.5 3.5) (thickness 0.8) bold) (justify left bottom))
   )
   (text "Bypass capacitor values taken directly from IC datasheet"
@@
     (effects (font (size 1.27 1.27)) (justify left bottom))
   )
+  (text "M2" (at 321.31 226.06 0)
+    (effects (font (size 1.5 1.5) (thickness 0.8) bold) (justify left bottom))
+  )
   (text "CL = 2*(CL0-Cs) = 2*(10-5) pF = 10 pF" (at 72.39 85.09 0)
     (effects (font (size 1.26 1.26)) (justify left bottom))
@@
     (effects (font (size 1.27 1.27)) (justify left bottom))
   )
-  (label "+IN" (at 106.68 200.66 0)
+  (label "IN+" (at 106.68 200.66 0)
     (effects (font (size 1.27 1.27)) (justify left bottom))
   )
@@
     (effects (font (size 0.4 0.4)) (justify left bottom))
   )
-  (label "-IN" (at 106.68 205.74 0)
+  (label "IN-" (at 106.68 205.74 0)
     (effects (font (size 1.27 1.27)) (justify left bottom))
   )
@@
     (pin "1")
   )
+  (symbol (lib_id "Mechanical:MountingHole") (at 326.39 218.44 0) (unit 1)
+    (in_bom yes) (on_board yes) (fields_autoplaced)
+    (property "Reference" "H4" (id 0) (at 328.93 217.1699 0)
+      (effects (font (size 1.27 1.27)) (justify left))
+    )
+    (property "Value" "MountingHole" (id 1) (at 328.93 219.7099 0)
+      (effects (font (size 1.27 1.27)) (justify left))
+    )
+    (property "Footprint" "MountingHole:MountingHole_2.2mm_M2" (id 2) (at 326.39 218.44 0)
+      (effects (font (size 1.27 1.27)) hide)
+    )
+    (property "Datasheet" "~" (id 3) (at 326.39 218.44 0)
+      (effects (font (size 1.27 1.27)) hide)
+    )
+  )
   (symbol (lib_id "Device:LED") (at 236.22 76.2 180) (unit 1)
     (in_bom yes) (on_board yes)
@@
     (pin "1")
     (pin "2")
+  )
+  (symbol (lib_id "Mechanical:MountingHole") (at 326.39 199.39 0) (unit 1)
+    (in_bom yes) (on_board yes) (fields_autoplaced)
+    (property "Reference" "H1" (id 0) (at 328.93 198.1199 0)
+      (effects (font (size 1.27 1.27)) (justify left))
+    )
+    (property "Value" "MountingHole" (id 1) (at 328.93 200.6599 0)
+      (effects (font (size 1.27 1.27)) (justify left))
+    )
+    (property "Footprint" "MountingHole:MountingHole_2.2mm_M2" (id 2) (at 326.39 199.39 0)
+      (effects (font (size 1.27 1.27)) hide)
+    )
+    (property "Datasheet" "~" (id 3) (at 326.39 199.39 0)
+      (effects (font (size 1.27 1.27)) hide)
+    )
   )
   (symbol (lib_id "power:+3.3VA") (at 217.17 46.99 0) (unit 1)
@@
     (pin "1")
     (pin "2")
+  )
+  (symbol (lib_id "Mechanical:MountingHole") (at 326.39 212.09 0) (unit 1)
+    (in_bom yes) (on_board yes) (fields_autoplaced)
+    (property "Reference" "H3" (id 0) (at 328.93 210.8199 0)
+      (effects (font (size 1.27 1.27)) (justify left))
+    )
+    (property "Value" "MountingHole" (id 1) (at 328.93 213.3599 0)
+      (effects (font (size 1.27 1.27)) (justify left))
+    )
+    (property "Footprint" "MountingHole:MountingHole_2.2mm_M2" (id 2) (at 326.39 212.09 0)
+      (effects (font (size 1.27 1.27)) hide)
+    )
+    (property "Datasheet" "~" (id 3) (at 326.39 212.09 0)
+      (effects (font (size 1.27 1.27)) hide)
+    )
   )
   (symbol (lib_id "power:GND") (at 336.55 160.02 0) (unit 1)
@@
     (pin "2")
   )
+  (symbol (lib_id "Mechanical:MountingHole") (at 326.39 205.74 0) (unit 1)
+    (in_bom yes) (on_board yes) (fields_autoplaced)
+    (property "Reference" "H2" (id 0) (at 328.93 204.4699 0)
+      (effects (font (size 1.27 1.27)) (justify left))
+    )
+    (property "Value" "MountingHole" (id 1) (at 328.93 207.0099 0)
+      (effects (font (size 1.27 1.27)) (justify left))
+    )
+    (property "Footprint" "MountingHole:MountingHole_2.2mm_M2" (id 2) (at 326.39 205.74 0)
+      (effects (font (size 1.27 1.27)) hide)
+    )
+    (property "Datasheet" "~" (id 3) (at 326.39 205.74 0)
+      (effects (font (size 1.27 1.27)) hide)
+    )
+  )
   (symbol (lib_id "Device:C") (at 87.63 236.22 0) (unit 1)
     (in_bom yes) (on_board yes) (fields_autoplaced)
@@
   (symbol (lib_id "power:GND") (at 363.22 125.73 0) (unit 1)
     (in_bom yes) (on_board yes) (fields_autoplaced)
-    (property "Reference" "#PWR0101" (id 0) (at 363.22 132.08 0)
+    (property "Reference" "#PWR028" (id 0) (at 363.22 132.08 0)
       (effects (font (size 1.27 1.27)) hide)
     )
@@
   (symbol (lib_id "power:GND") (at 146.05 85.09 0) (unit 1)
     (in_bom yes) (on_board yes) (fields_autoplaced)
-    (property "Reference" "#PWR0103" (id 0) (at 146.05 91.44 0)
+    (property "Reference" "#PWR07" (id 0) (at 146.05 91.44 0)
       (effects (font (size 1.27 1.27)) hide)
     )
@@
   (symbol (lib_id "power:GND") (at 153.67 241.3 0) (unit 1)
     (in_bom yes) (on_board yes) (fields_autoplaced)
-    (property "Reference" "#PWR07" (id 0) (at 153.67 247.65 0)
+    (property "Reference" "#PWR09" (id 0) (at 153.67 247.65 0)
       (effects (font (size 1.27 1.27)) hide)
     )
@@
   (symbol (lib_id "power:+5V") (at 358.14 111.76 0) (unit 1)
     (in_bom yes) (on_board yes) (fields_autoplaced)
-    (property "Reference" "#PWR0102" (id 0) (at 358.14 115.57 0)
+    (property "Reference" "#PWR027" (id 0) (at 358.14 115.57 0)
       (effects (font (size 1.27 1.27)) hide)
     )
@@
       (reference "#PWR06") (unit 1) (value "GND") (footprint "")
     )
-    (path "/851c3dcb-6946-4b9b-80b1-5c8fba1fdccb"
+    (path "/8081c97e-d308-4576-b4e6-ef99492c41c9"
       (reference "#PWR07") (unit 1) (value "GND") (footprint "")
     )
@@
       (reference "#PWR08") (unit 1) (value "+3.3V") (footprint "")
     )
+    (path "/851c3dcb-6946-4b9b-80b1-5c8fba1fdccb"
+      (reference "#PWR09") (unit 1) (value "GND") (footprint "")
+    )
     (path "/3e7d9861-6f20-434f-a5bc-fa93ba3d66ab"
       (reference "#PWR010") (unit 1) (value "+3.3V") (footprint "")
@@
       (reference "#PWR026") (unit 1) (value "GND") (footprint "")
     )
+    (path "/ec028ad3-bc24-474c-b113-d180e751ef90"
+      (reference "#PWR027") (unit 1) (value "+5V") (footprint "")
+    )
     (path "/7bed3991-a053-4cdf-bd1e-022feab5cce8"
-      (reference "#PWR0101") (unit 1) (value "GND") (footprint "")
-    )
-    (path "/ec028ad3-bc24-474c-b113-d180e751ef90"
-      (reference "#PWR0102") (unit 1) (value "+5V") (footprint "")
-    )
-    (path "/8081c97e-d308-4576-b4e6-ef99492c41c9"
-      (reference "#PWR0103") (unit 1) (value "GND") (footprint "")
+      (reference "#PWR028") (unit 1) (value "GND") (footprint "")
     )
     (path "/31891be7-3501-4833-81d8-aeb671487980"
@@
       (reference "FB1") (unit 1) (value "120R") (footprint "Inductor_SMD:L_0603_1608Metric")
     )
+    (path "/1653a934-bd12-47dc-9d67-283df9fc5bed"
+      (reference "H1") (unit 1) (value "MountingHole") (footprint "MountingHole:MountingHole_2.2mm_M2")
+    )
+    (path "/54e6013e-72eb-4766-ba6f-ede2c2d0fb16"
+      (reference "H2") (unit 1) (value "MountingHole") (footprint "MountingHole:MountingHole_2.2mm_M2")
+    )
+    (path "/445ef171-8048-4ec0-b7ed-9f50fb76ae7e"
+      (reference "H3") (unit 1) (value "MountingHole") (footprint "MountingHole:MountingHole_2.2mm_M2")
+    )
+    (path "/08a608d9-2e34-464c-b171-8c23997c8e4c"
+      (reference "H4") (unit 1) (value "MountingHole") (footprint "MountingHole:MountingHole_2.2mm_M2")
+    )
     (path "/93f9e328-4970-40f9-97a6-cad5c6e8b8f4"

Commit message: restored Octave algo script
Connections:
- net AD8232_LOD_N: now also U1.12 (LO+), U2.10 (PC2); no longer U1.11 (LO-), U2.9 (PC1)
- net AD8232_LOD_P: now also U1.11 (LO-), U2.9 (PC1); no longer U1.12 (LO+), U2.8 (PC0)
Changed lines of the file:
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@@
   (junction (at 342.9 46.99) (diameter 0) (color 0 0 0 0)
   )
+  (junction (at 214.63 152.4) (diameter 0) (color 0 0 0 0)
+  )
   (junction (at 87.63 231.14) (diameter 0) (color 0 0 0 0)
   )
@@
   )
   (junction (at 217.17 46.99) (diameter 0) (color 0 0 0 0)
+  )
+  (junction (at 339.09 46.99) (diameter 0) (color 0 0 0 0)
   )
   (no_connect (at 191.77 137.16))
@@
   (no_connect (at 323.85 134.62))
   (no_connect (at 227.33 121.92))
+  (no_connect (at 191.77 106.68))
   (no_connect (at 323.85 109.22))
   (no_connect (at 227.33 86.36))
@@
   (no_connect (at 323.85 127))
   (no_connect (at 363.22 121.92))
-  (no_connect (at 191.77 111.76))
   (no_connect (at 227.33 114.3))
   (no_connect (at 227.33 142.24))
@@
     (stroke (width 0) (type default) (color 0 0 0 0))
   )
+  (wire (pts (xy 167.64 111.76) (xy 167.64 171.45))
+    (stroke (width 0) (type default) (color 0 0 0 0))
+  )
   (wire (pts (xy 261.62 119.38) (xy 259.08 119.38))
     (stroke (width 0) (type default) (color 0 0 0 0))
@@
     (stroke (width 0) (type default) (color 0 0 0 0))
   )
-  (wire (pts (xy 167.64 106.68) (xy 191.77 106.68))
-    (stroke (width 0) (type default) (color 0 0 0 0))
-  )
   (wire (pts (xy 323.85 104.14) (xy 261.62 104.14))
     (stroke (width 0) (type default) (color 0 0 0 0))
@@
     (stroke (width 0) (type default) (color 0 0 0 0))
   )
+  (wire (pts (xy 154.94 241.3) (xy 153.67 241.3))
+    (stroke (width 0) (type default) (color 0 0 0 0))
+  )
   (wire (pts (xy 92.71 101.6) (xy 92.71 104.14))
     (stroke (width 0) (type default) (color 0 0 0 0))
@@
     (stroke (width 0) (type default) (color 0 0 0 0))
   )
-  (wire (pts (xy 167.64 106.68) (xy 167.64 171.45))
-    (stroke (width 0) (type default) (color 0 0 0 0))
-  )
   (polyline (pts (xy 287.02 163.83) (xy 137.16 163.83))
     (stroke (width 0) (type default) (color 0 0 0 0))
@@
   )
   (wire (pts (xy 87.63 88.9) (xy 87.63 104.14))
+    (stroke (width 0) (type default) (color 0 0 0 0))
+  )
+  (wire (pts (xy 167.64 111.76) (xy 191.77 111.76))
     (stroke (width 0) (type default) (color 0 0 0 0))
   )
@@
     (effects (font (size 1.27 1.27)) (justify left bottom))
   )
-  (label "AD8232_LOD_N" (at 170.18 109.22 0)
+  (label "AD8232_LOD_P" (at 171.45 109.22 0)
+    (effects (font (size 1.27 1.27)) (justify left bottom))
+  )
+  (label "~SDN" (at 154.94 251.46 0)
     (effects (font (size 1.27 1.27)) (justify left bottom))
   )
@@
   )
   (label "LED" (at 227.33 76.2 0)
+    (effects (font (size 1.27 1.27)) (justify left bottom))
+  )
+  (label "AC{slash}~DC" (at 153.67 241.3 0)
+    (effects (font (size 1.27 1.27)) (justify left bottom))
+  )
+  (label "FR" (at 154.94 236.22 0)
     (effects (font (size 1.27 1.27)) (justify left bottom))
   )
@@
     (effects (font (size 1.27 1.27)) (justify left bottom))
   )
-  (label "AD8232_LOD_P" (at 170.18 106.68 0)
+  (label "AD8232_LOD_N" (at 171.45 111.76 0)
     (effects (font (size 1.27 1.27)) (justify left bottom))
   )
@@
     (pin "1")
     (pin "2")
+  )
+  (symbol (lib_id "power:PWR_FLAG") (at 214.63 152.4 180) (unit 1)
+    (in_bom yes) (on_board yes) (fields_autoplaced)
+    (property "Reference" "#FLG0102" (id 0) (at 214.63 154.305 0)
+      (effects (font (size 1.27 1.27)) hide)
+    )
+    (property "Value" "PWR_FLAG" (id 1) (at 217.17 153.6699 0)
+      (effects (font (size 1.27 1.27)) (justify right))
+    )
+    (property "Footprint" "" (id 2) (at 214.63 152.4 0)
+      (effects (font (size 1.27 1.27)) hide)
+    )
+    (property "Datasheet" "~" (id 3) (at 214.63 152.4 0)
+      (effects (font (size 1.27 1.27)) hide)
+    )
+    (pin "1")
   )
   (symbol (lib_id "Mechanical:MountingHole") (at 326.39 212.09 0) (unit 1)
@@
     (pin "1")
   )
-  (symbol (lib_id "power:GND") (at 153.67 241.3 0) (unit 1)
-    (in_bom yes) (on_board yes) (fields_autoplaced)
-    (property "Reference" "#PWR09" (id 0) (at 153.67 247.65 0)
-      (effects (font (size 1.27 1.27)) hide)
-    )
-    (property "Value" "GND" (id 1) (at 153.67 246.38 0)
-      (effects (font (size 1.27 1.27)) hide)
-    )
-    (property "Footprint" "" (id 2) (at 153.67 241.3 0)
-      (effects (font (size 1.27 1.27)) hide)
-    )
-    (property "Datasheet" "" (id 3) (at 153.67 241.3 0)
+  (symbol (lib_id "power:GND") (at 154.94 241.3 0) (unit 1)
+    (in_bom yes) (on_board yes) (fields_autoplaced)
+    (property "Reference" "#PWR09" (id 0) (at 154.94 247.65 0)
+      (effects (font (size 1.27 1.27)) hide)
+    )
+    (property "Value" "GND" (id 1) (at 154.94 246.38 0)
+      (effects (font (size 1.27 1.27)) hide)
+    )
+    (property "Footprint" "" (id 2) (at 154.94 241.3 0)
+      (effects (font (size 1.27 1.27)) hide)
+    )
+    (property "Datasheet" "" (id 3) (at 154.94 241.3 0)
       (effects (font (size 1.27 1.27)) hide)
     )
@@
     (pin "2")
   )
+  (symbol (lib_id "power:PWR_FLAG") (at 339.09 46.99 0) (unit 1)
+    (in_bom yes) (on_board yes) (fields_autoplaced)
+    (property "Reference" "#FLG0101" (id 0) (at 339.09 45.085 0)
+      (effects (font (size 1.27 1.27)) hide)
+    )
+    (property "Value" "PWR_FLAG" (id 1) (at 339.09 41.91 0))
+    (property "Footprint" "" (id 2) (at 339.09 46.99 0)
+      (effects (font (size 1.27 1.27)) hide)
+    )
+    (property "Datasheet" "~" (id 3) (at 339.09 46.99 0)
+      (effects (font (size 1.27 1.27)) hide)
+    )
+    (pin "1")
+  )
   (symbol (lib_id "Device:R") (at 87.63 256.54 0) (mirror y) (unit 1)
     (in_bom yes) (on_board yes) (fields_autoplaced)
@@
       (reference "#FLG02") (unit 1) (value "PWR_FLAG") (footprint "")
     )
+    (path "/c7105d6e-bc82-4bb9-99fa-318d0dc2fa2c"
+      (reference "#FLG0101") (unit 1) (value "PWR_FLAG") (footprint "")
+    )
+    (path "/41566288-d122-4009-8da0-36044064dd4a"
+      (reference "#FLG0102") (unit 1) (value "PWR_FLAG") (footprint "")
+    )
     (path "/e3a4fcd0-9005-4f3c-8e03-7eaa188822ab"
