File: pcb/pcb.kicad_pcb (KiCad board)
At the start: 4 copper layers, 61 x 33.1 mm, 57 parts, among them J1 PJ-320D-A, J2 Conn_01x02_Male, J3 Conn_01x04_Male, J4 105133-0011, SW1 PCM12SMTR, U1 AD8232, U2 STM32F334R8T6, U3 CP2102N-A02-GQFN20R, Y1 16MHz

Commit message: pcb finished
Parts:
- C15, C6: value 330n -> 3300p
- R13, R14: value 10Meg -> 9.09Meg
- R15: value 1.4Meg -> 1.27Meg
- R2, R4: value 1Meg -> 287k
- moved R18 31.5 mm to (59.5, 45.3)
- moved C21 31.4 mm to (57.5, 45.7)
- moved C5 31.3 mm to (62.5, 37.3)
- moved C1 31.2 mm to (96.9, 38.2)
- moved C11 31.2 mm to (80.9, 31.8)
- moved C14 31.2 mm to (76.7, 42.8)
- moved C15 31.2 mm to (99.1, 24.3)
- moved C17 31.2 mm to (63.6, 40.4)
- moved C18 31.2 mm to (63.6, 43.5)
- moved C22 31.2 mm to (54.6, 47.3)
- moved C3 31.2 mm to (93.7, 36.4)
- moved C4 31.2 mm to (92.4, 33.3)
- moved D1 31.2 mm to (72.4, 44.2)
- moved FB1 31.2 mm to (66.7, 42.1)
- moved H2 31.2 mm to (103.4, 50.1)
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Connections:
- U2 pad 17: /USART2_RX -> unconnected-(U2-Pad17)
- U3 pad 18: /USART2_RX -> unconnected-(U3-Pad18)
Routing:
- net +3.3V: track 14.0 -> 160.4 mm, vias 0 -> 13
- net +5V: track 0.00 -> 22.4 mm, vias 0 -> 2
- net GND: track 48.7 -> 69.2 mm, vias 6 -> 19
- net /NRST: track 0.00 -> 10.5 mm, vias 0 -> 2
- net /USART2_TX: track 0.00 -> 9.78 mm
- net /USB_D+: track 0.00 -> 8.38 mm, vias 0 -> 2
- net /USB_D-: track 0.00 -> 8.10 mm
- net +3.3VA: track 2.33 -> 9.58 mm, vias 0 -> 2
- net Net-(R18-Pad2): track 0.00 -> 2.71 mm
- net /IN-: track 5.37 -> 6.89 mm
- net /ADC1_IN1: track 64.2 -> 63.5 mm
Other:
- copper layers 4 -> 2
- board text added: "06/23"
- board text added: "3V3"
- board text added: "BOOT"
- board text added: "GND"
- board text added: "HR"
- board text added: "JACK"
- board text added: "OUT"
- board text added: "PWR"
- board text added: "Rev: 0.1"
- board text added: "SIG"
- board text added: "SWD"
- board text added: "TCK"
- board text added: "TMS"
- board text added: "USB"
