File: pcb/pcb.kicad_sch (KiCad schematic)
At the start: 56 parts, among them J1 PJ-320D-A, J2 Conn_01x02_Male, J3 Conn_01x04_Male, J4 105133-0011, SW1 PCM12SMTR, U1 AD8232, U2 STM32F334R8T6, U3 CP2102N-A02-GQFN20R, Y1 16MHz

Commit message: pcb finished
Parts:
- C15, C6: value 330n -> 3300p
- R13, R14: value 10Meg -> 9.09Meg
- R15: value 1.4Meg -> 1.27Meg
- R2, R4: value 1Meg -> 287k
Connections:
- net USART2_RX: no longer names the net of U3.18 (TXD)
- net USART2_RX: no longer U2.17 (PA3)
- no-connect marks 54 -> 56
Changed lines of the file:
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@@
   (no_connect (at 191.77 134.62))
   (no_connect (at 227.33 129.54))
+  (no_connect (at 323.85 101.6))
   (no_connect (at 227.33 111.76))
   (no_connect (at 191.77 101.6))
@@
   (no_connect (at 191.77 116.84))
   (no_connect (at 227.33 91.44))
+  (no_connect (at 227.33 71.12))
   (no_connect (at 227.33 139.7))
   (no_connect (at 323.85 134.62))
@@
     (stroke (width 0) (type default) (color 0 0 0 0))
   )
-  (wire (pts (xy 264.16 101.6) (xy 323.85 101.6))
-    (stroke (width 0) (type default) (color 0 0 0 0))
-  )
   (wire (pts (xy 207.01 152.4) (xy 209.55 152.4))
     (stroke (width 0) (type default) (color 0 0 0 0))
   )
-  (wire (pts (xy 227.33 71.12) (xy 264.16 71.12))
-    (stroke (width 0) (type default) (color 0 0 0 0))
-  )
   (wire (pts (xy 99.06 176.53) (xy 195.58 176.53))
     (stroke (width 0) (type default) (color 0 0 0 0))
@@
   )
   (wire (pts (xy 157.48 171.45) (xy 157.48 205.74))
-    (stroke (width 0) (type default) (color 0 0 0 0))
-  )
-  (wire (pts (xy 264.16 71.12) (xy 264.16 101.6))
     (stroke (width 0) (type default) (color 0 0 0 0))
   )
@@
   )
   (label "TMS" (at 233.68 96.52 0)
-    (effects (font (size 1.27 1.27)) (justify left bottom))
-  )
-  (label "USART2_RX" (at 227.33 71.12 0)
     (effects (font (size 1.27 1.27)) (justify left bottom))
   )
@@
       (effects (font (size 1.27 1.27)) (justify right))
     )
-    (property "Value" "10Meg" (id 1) (at 187.96 201.9299 0)
+    (property "Value" "9.09Meg" (id 1) (at 187.96 201.9299 0)
       (effects (font (size 1.27 1.27)) (justify right))
     )
@@
     (in_bom yes) (on_board yes) (fields_autoplaced)
     (property "Reference" "R2" (id 0) (at 67.31 224.79 90))
-    (property "Value" "1Meg" (id 1) (at 67.31 227.33 90))
+    (property "Value" "287k" (id 1) (at 67.31 227.33 90))
     (property "Footprint" "Resistor_SMD:R_0603_1608Metric" (id 2) (at 67.31 232.918 90)
       (effects (font (size 1.27 1.27)) hide)
@@
     (in_bom yes) (on_board yes) (fields_autoplaced)
     (property "Reference" "R13" (id 0) (at 177.8 199.39 90))
-    (property "Value" "10Meg" (id 1) (at 177.8 201.93 90))
+    (property "Value" "9.09Meg" (id 1) (at 177.8 201.93 90))
     (property "Footprint" "Resistor_SMD:R_0603_1608Metric" (id 2) (at 177.8 207.518 90)
       (effects (font (size 1.27 1.27)) hide)
@@
     (in_bom yes) (on_board yes) (fields_autoplaced)
     (property "Reference" "C6" (id 0) (at 133.35 179.07 90))
-    (property "Value" "330n" (id 1) (at 133.35 181.61 90))
+    (property "Value" "3300p" (id 1) (at 133.35 181.61 90))
     (property "Footprint" "Capacitor_SMD:C_0402_1005Metric" (id 2) (at 137.16 185.7248 0)
       (effects (font (size 1.27 1.27)) hide)
@@
       (effects (font (size 1.27 1.27)) (justify right))
     )
-    (property "Value" "1.4Meg" (id 1) (at 187.96 212.0899 0)
+    (property "Value" "1.27Meg" (id 1) (at 187.96 212.0899 0)
       (effects (font (size 1.27 1.27)) (justify right))
     )
@@
       (effects (font (size 1.27 1.27)) (justify right))
     )
-    (property "Value" "330n" (id 1) (at 199.39 223.5199 0)
+    (property "Value" "3300p" (id 1) (at 199.39 223.5199 0)
       (effects (font (size 1.27 1.27)) (justify right))
     )
@@
     (in_bom yes) (on_board yes) (fields_autoplaced)
     (property "Reference" "R4" (id 0) (at 81.28 224.79 90))
-    (property "Value" "1Meg" (id 1) (at 81.28 227.33 90))
+    (property "Value" "287k" (id 1) (at 81.28 227.33 90))
     (property "Footprint" "Resistor_SMD:R_0603_1608Metric" (id 2) (at 81.28 232.918 90)
       (effects (font (size 1.27 1.27)) hide)
@@
     )
     (path "/4d3a038d-b46c-4adc-b4c6-3ff9e9a9ac09"
-      (reference "C6") (unit 1) (value "330n") (footprint "Capacitor_SMD:C_0402_1005Metric")
+      (reference "C6") (unit 1) (value "3300p") (footprint "Capacitor_SMD:C_0402_1005Metric")
     )
     (path "/e79a7b0f-c00e-40e7-857b-e8c63fecb6ab"
@@
     )
     (path "/920a9f53-4c01-447a-a0dc-cc23ac170431"
-      (reference "C15") (unit 1) (value "330n") (footprint "Capacitor_SMD:C_0402_1005Metric")
+      (reference "C15") (unit 1) (value "3300p") (footprint "Capacitor_SMD:C_0402_1005Metric")
     )
     (path "/d54e3e70-358f-4ba4-ab50-703cc07bca61"
@@
     )
     (path "/148d136e-87a7-4ee9-ad60-44e1e38b48fd"
-      (reference "R2") (unit 1) (value "1Meg") (footprint "Resistor_SMD:R_0603_1608Metric")
+      (reference "R2") (unit 1) (value "287k") (footprint "Resistor_SMD:R_0603_1608Metric")
     )
     (path "/f29f513d-1979-42b8-94ce-181029c0da32"
@@
     )
     (path "/d0843e75-a712-4ca5-9518-f69926846b86"
-      (reference "R4") (unit 1) (value "1Meg") (footprint "Resistor_SMD:R_0603_1608Metric")
+      (reference "R4") (unit 1) (value "287k") (footprint "Resistor_SMD:R_0603_1608Metric")
     )
     (path "/134b913c-9762-4c9f-b452-b78e56bfa844"
@@
     )
     (path "/2408c4f0-3c09-4661-88e4-94885ab1bd87"
-      (reference "R13") (unit 1) (value "10Meg") (footprint "Resistor_SMD:R_0603_1608Metric")
+      (reference "R13") (unit 1) (value "9.09Meg") (footprint "Resistor_SMD:R_0603_1608Metric")
     )
     (path "/0fee8e1a-1b82-4e63-90fd-d7e9fa01a515"
-      (reference "R14") (unit 1) (value "10Meg") (footprint "Resistor_SMD:R_0603_1608Metric")
+      (reference "R14") (unit 1) (value "9.09Meg") (footprint "Resistor_SMD:R_0603_1608Metric")
     )
     (path "/524c1fba-d755-4cdf-aef7-ac104b7dc5b5"
-      (reference "R15") (unit 1) (value "1.4Meg") (footprint "Resistor_SMD:R_0603_1608Metric")
+      (reference "R15") (unit 1) (value "1.27Meg") (footprint "Resistor_SMD:R_0603_1608Metric")
     )
     (path "/54403a77-908f-4e67-9319-8a2d9517b149"
